File: hw/ictester.kicad_sch (KiCad schematic)
At the start: 70 parts, among them J1 Conn_01x12_Pin, J2 Conn_01x12_Pin, J3 Conn_01x01_Pin, J4 Conn_01x01_Pin, J6 Conn_01x06_Pin, J7 Conn_01x04_Pin, J8 Conn_02x05_Odd_Even, J9 USB_B_Micro, U1 ATmega1284-A, U2 CP2102N-Axx-xQFN28, U3 CDSOT236-0504C, U4 MAX14662, U5 MAX14662, U6 MAX14662, U7 MAX14662, U8 MAX14662, U9 ZIF24, Y1 20MHz

Commit message: h/w update
Parts:
- added C18: 100n, Capacitor_SMD:C_0805_2012Metric_Pad1.18x1.45mm_HandSolder, symbol Device:C_Small
- C7: value 10n -> 100n
- C8: value C_Polarized -> 10u
Connections:
- net +5V: now also C18.2; no longer U1.29 (AREF)
- net GND: now also C18.1
- no-connect marks 25 -> 26
Other:
- note added: "all 4k7"
- note removed: "4k7"
- company: (none) -> https://mera400.pl
- title: (none) -> Logic IC tester
- moved on the sheet: R1

Commit message: hw update
Connections:
- net +5V: now also J8.4 (Pin_4), J8.6 (Pin_6)
- net GND: no longer J8.4 (Pin_4), J8.6 (Pin_6)
- net at J6.6 (Pin_6): now also C1.1, U2.6 (VDD)
- net MISO renamed ZIF23
- net MOSI renamed ZIF22
- net SCK renamed ZIF24
- no-connect marks 26 -> 25
Other:
- moved on the sheet: C10, C12, C14, C17, C18, C2, C4, C6, C7, C9, J3, J4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

Commit message: H/W v3
Parts:
- removed C1, C13, C18: 100n, Capacitor_SMD:C_0805_2012Metric_Pad1.18x1.45mm_HandSolder, symbol Device:C_Small
- removed C15, C16, C17, C9: 470p, Capacitor_SMD:C_0805_2012Metric_Pad1.18x1.45mm_HandSolder, symbol Device:C_Small
- removed C2: 22p, Capacitor_SMD:C_0805_2012Metric_Pad1.18x1.45mm_HandSolder, symbol Device:C_Small
- removed C8: 10u, Capacitor_Tantalum_SMD:CP_EIA-3528-21_Kemet-B_Pad1.50x2.35mm_HandSolder, symbol Device:C_Polarized
- removed H1, H2, H3, H4: MountingHole_Pad, MountingHole:MountingHole_3.2mm_M3_DIN965_Pad_TopBottom, symbol Mechanical:MountingHole_Pad
- removed J6: Conn_01x06_Pin, Connector_PinHeader_2.54mm:PinHeader_1x06_P2.54mm_Vertical, symbol Connector:Conn_01x06_Pin
- removed J7: Conn_01x04_Pin, Connector_PinHeader_2.54mm:PinHeader_1x04_P2.54mm_Vertical, symbol Connector:Conn_01x04_Pin
- removed J8: Conn_02x05_Odd_Even, Connector_PinHeader_2.54mm:PinHeader_2x05_P2.54mm_Vertical, symbol Connector_Generic:Conn_02x05_Odd_Even
- removed J9: USB_B_Micro, Connector_USB:USB_Micro-B_Amphenol_10104110_Horizontal, symbol Connector:USB_B_Micro
- removed JP1: Jumper_2_Open, Connector_PinHeader_2.54mm:PinHeader_1x02_P2.54mm_Vertical, symbol Jumper:Jumper_2_Open
- removed LED1: Inolux_IN-PI554FCH, LED_SMD:LED_Inolux_IN-PI554FCH_PLCC4_5.0x5.0mm_P3.2mm, symbol LED:Inolux_IN-PI554FCH
- removed R1: 10k, Resistor_SMD:R_0805_2012Metric_Pad1.20x1.40mm_HandSolder, symbol Device:R_Small
- removed R12, R2, R22, R23, R24, R3, R4: 4k7, Resistor_SMD:R_0805_2012Metric_Pad1.20x1.40mm_HandSolder, symbol Device:R_Small
- removed U1: ATmega1284-A, Package_QFP:TQFP-44_10x10mm_P0.8mm, symbol MCU_Microchip_ATmega:ATmega1284-A
- removed U2: CP2102N-Axx-xQFN28, Package_DFN_QFN:QFN-28-1EP_5x5mm_P0.5mm_EP3.35x3.35mm, symbol Interface_USB:CP2102N-Axx-xQFN28
- removed U3: CDSOT236-0504C, Package_TO_SOT_SMD:SOT-23-6, symbol Power_Protection:CDSOT236-0504C
- removed U8: MAX14662, Package_DFN_QFN:QFN-28-1EP_4x4mm_P0.4mm_EP2.6x2.6mm, symbol ictester:MAX14662
- removed Y1: 20MHz, Crystal:Crystal_SMD_Abracon_ABM3C-4Pin_5.0x3.2mm, symbol Device:Crystal_GND24_Small
- added R13, R14, R15: 4k7, Resistor_SMD:R_0805_2012Metric_Pad1.20x1.40mm_HandSolder, symbol Device:R_Small
- added U3: MAX14662, Package_DFN_QFN:QFN-28-1EP_4x4mm_P0.4mm_EP2.6x2.6mm, symbol ictester:MAX14662
- C3, C6, C7: value 100n -> 470p
- C4: value 22p -> 100n
- C5: value 1u -> 470p
- renumbered C14 to C1, C12 to C2, C10 to C8, C11 to C9, J4 to J1, J1 to J3, J3 to J4, R21 to R1, R20 to R10, R29 to R11, R28 to R12, R13 to R16, R14 to R17, R17 to R18, R6 to R19, R25 to R2, R7 to R20, R8 to R21, R9 to R22, R10 to R23, R11 to R24, R26 to R3, R27 to R4, R16 to R6, R15 to R7, R18 to R8, R19 to R9, U7 to U1, U6 to U2, U9 to U4, U4 to U6
Connections:
- net +5V: now also C4.1, R5.2, R13.1, R14.1, R15.1, U3.26 (VCC), U3.28 (DOUT/AD1); no longer C3.1, C5.1, C6.2, C7.2, R5.1, U1.23 (~{CS}/AD0)
- net GND: now also C4.2, C5.1, U1.23 (~{CS}/AD0), U3.1 (SPI/~{I2C}), U3.11 (GND), U3.23 (~{CS}/AD0), U3.25 (GND), U3.29 (GND); no longer C3.2, C4.1, C5.2, C6.1, C7.1, U1.7 (A6), U2.2 (A1), U2.5 (A4), U5.17 (B5), U5.18 (B4), U6.2 (A1)
- net SCL2: now also U3.24 (SCLK/SCL); no longer R5.2
- net SDA2: now also U3.27 (DIN/SDA)
- net ZIF1: now also U6.2 (A1); no longer U6.20 (B2), U6.21 (B1)
- net ZIF10: now also U5.8 (A7), U5.9 (A8); no longer U2.17 (B5), U2.18 (B4)
- net ZIF11: now also U2.4 (A3); no longer U2.19 (B3)
- net ZIF12: now also U2.2 (A1), U2.3 (A2); no longer U2.20 (B2), U2.21 (B1)
- net ZIF13: now also U2.9 (A8); no longer U2.14 (B8)
- net ZIF14: now also U2.8 (A7); no longer U2.15 (B7)
- net ZIF15: now also U2.7 (A6); no longer U2.16 (B6)
- net ZIF16: now also U2.6 (A5); no longer U1.21 (B1)
- net ZIF17: now also U2.5 (A4); no longer U1.20 (B2)
- net ZIF18: now also U1.14 (B8); no longer U1.19 (B3)
- net ZIF19: now also U1.15 (B7); no longer U1.18 (B4)
- net ZIF2: now also U6.3 (A2); no longer U6.19 (B3)
- net ZIF20: now also U3.7 (A6); no longer U1.15 (B7)
- net ZIF21: now also U1.18 (B4), U3.5 (A4), U3.6 (A5); no longer U1.14 (B8)
- net ZIF22: now also U3.3 (A2), U3.4 (A3)
- net ZIF23: now also U3.2 (A1)
- net ZIF24: now also U1.19 (B3), U1.20 (B2), U1.21 (B1)
- net ZIF3: now also U6.4 (A3); no longer U6.18 (B4)
- net ZIF4: now also U6.5 (A4), U6.6 (A5); no longer U6.16 (B6), U6.17 (B5)
- net ZIF5: now also U6.7 (A6), U6.8 (A7); no longer U6.14 (B8), U6.15 (B7)
- net ZIF6: now also U6.9 (A8), U3.15 (B7); no longer U5.8 (A7), U5.9 (A8)
- net ZIF7: now also U5.2 (A1), U3.14 (B8); no longer U5.6 (A5), U5.7 (A6)
- net ZIF9: now also U5.6 (A5), U5.7 (A6); no longer U5.2 (A1)
- net at U1.9 (A8): now also R4.1
- net at R19.1: now also U6.21 (B1); no longer U6.3 (A2)
- net at R20.1: now also U6.20 (B2); no longer U6.4 (A3)
- net at R21.1: now also U6.19 (B3); no longer U6.5 (A4)
- net at R22.1: now also U6.18 (B4); no longer U6.6 (A5)
- net at R23.1: now also U6.15 (B7); no longer U6.8 (A7)
- net at R24.1: now also U6.14 (B8); no longer U5.14 (B8)
- net at U5.15 (B7): now also R18.1
- net VDUT: now reaches U5.16 (B6)
- net VDUT: now also U1.3 (A2), U5.20 (B2), U6.16 (B6), U6.17 (B5)
- net at R16.1: now also U5.19 (B3); no longer U5.20 (B2)
- net at R17.1: now also U5.17 (B5); no longer U5.21 (B1)
- net at R3.1: now also U1.8 (A7); no longer U1.5 (A4)
- net at R8.1: now also U2.18 (B4); no longer U2.7 (A6)
- net at R11.1: now also U2.15 (B7); no longer U1.2 (A1)
- net at R12.1: now also U2.14 (B8); no longer U1.3 (A2)
- net at U1.4 (A3): now also R1.1; no longer R4.1
- net at R10.1: now also U2.16 (B6); no longer U2.9 (A8)
- net at R7.1: now also U2.19 (B3); no longer U2.3 (A2)
- net at R6.1: now also U2.21 (B1); no longer U2.4 (A3)
- net at R9.1: now also U2.17 (B5); no longer U2.8 (A7)
- removed net +5VD: U5.19 (B3), U6.7 (A6), U6.9 (A8)
- net ~{RESET} renamed ~{SD}
- net ~{SD}: now also U3.22 (~{SD})
- new net: C3.1, U3.8 (A7)
- new net: C3.2, R5.1, U3.9 (A8)
- new net: C7.1, R15.2, U3.17 (B5)
- new net: C7.2, U3.16 (B6)
- new net: C5.2, C6.2, U3.18 (B4), U3.20 (B2)
- new net: R14.2, U3.19 (B3)
- new net: C6.1, R13.2, U3.21 (B1)
- new net GNDUT: U1.2 (A1), U1.5 (A4), U1.7 (A6), U2.20 (B2), U5.14 (B8), U5.18 (B4), U5.21 (B1)
- no-connect marks 25 -> 0
Other:
- added sheet CURRENT (isense.kicad_sch)
- added sheet MCU (mcu.kicad_sch)
- added sheet USB (usb.kicad_sch)
- note added: "4k7"
- note added: "A0"
- note added: "A1"
- note added: "A2"
- note added: "B0"
- note added: "B1"
- note removed: "all 4k7"
- moved on the sheet: C1, C2, C8, C9, J1, J2, J3, J4, R1, R10, R11, R12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
