File: hw/mcu.kicad_sch (KiCad schematic)
At the start: 28 parts, among them J5 Conn_02x05_Odd_Even, U7 74LVC1G07, U8 ATmega1284-A, Y1 20MHz

Commit message: improve oscillator grounding
Parts:
- added NT1: NetTie_2, NetTie:NetTie-2_SMD_Pad0.5mm, symbol Device:NetTie_2
Connections:
- net GND: now also NT1.1; no longer C10.2, C11.1, Y1.2, Y1.4
- new net GNDOSC: C10.2, C11.1, NT1.2, Y1.2, Y1.4
Changed lines of the file:
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@@
 	(wire
 		(pts
+			(xy 41.91 71.12) (xy 41.91 69.85)
+		)
+		(stroke
+			(width 0)
+			(type default)
+		)
+	)
+	(wire
+		(pts
 			(xy 210.82 111.76) (xy 222.25 111.76)
 		)
@@
 	(wire
 		(pts
-			(xy 52.07 60.96) (xy 52.07 64.77)
+			(xy 52.07 60.96) (xy 52.07 69.85)
 		)
 		(stroke
@@
 	(wire
 		(pts
+			(xy 41.91 69.85) (xy 43.18 69.85)
+		)
+		(stroke
+			(width 0)
+			(type default)
+		)
+	)
+	(wire
+		(pts
 			(xy 143.51 46.99) (xy 143.51 63.5)
 		)
@@
 	(wire
 		(pts
+			(xy 48.26 69.85) (xy 52.07 69.85)
+		)
+		(stroke
+			(width 0)
+			(type default)
+		)
+	)
+	(wire
+		(pts
 			(xy 139.7 124.46) (xy 153.67 124.46)
 		)
@@
 		)
 	)
+	(label "GNDOSC"
+		(at 52.07 69.85 0)
+		(effects
+			(font
+				(size 1.27 1.27)
+			)
+			(justify left bottom)
+		)
+	)
 	(global_label "ZIF17"
 		(shape bidirectional)
@@
 	(symbol
 		(lib_id "power:GND")
-		(at 52.07 64.77 0)
+		(at 41.91 71.12 0)
 		(unit 1)
 		(exclude_from_sim no)
@@
 		(dnp no)
 		(property "Reference" "#PWR046"
-			(at 52.07 71.12 0)
+			(at 41.91 77.47 0)
 			(effects
 				(font
@@
 		)
 		(property "Value" "GND"
-			(at 52.705 68.58 0)
+			(at 42.545 74.93 0)
 			(effects
 				(font
@@
 		)
 		(property "Footprint" ""
-			(at 52.07 64.77 0)
+			(at 41.91 71.12 0)
 			(effects
 				(font
@@
 		)
 		(property "Datasheet" ""
-			(at 52.07 64.77 0)
+			(at 41.91 71.12 0)
 			(effects
 				(font
@@
 		)
 		(property "Description" "Power symbol creates a global label with name \"GND\" , ground"
-			(at 52.07 64.77 0)
+			(at 41.91 71.12 0)
 			(effects
 				(font
@@
 					(unit 1)
 				)
+			)
+		)
+	)
+	(symbol
+		(lib_id "Device:NetTie_2")
+		(at 45.72 69.85 0)
+		(unit 1)
+		(exclude_from_sim no)
+		(in_bom no)
+		(on_board yes)
+		(dnp no)
+		(fields_autoplaced yes)
+		(property "Reference" "NT1"
+			(at 45.72 64.77 0)
+			(effects
+				(font
+					(size 1.27 1.27)
+				)
+			)
+		)
+		(property "Value" "NetTie_2"
+			(at 45.72 67.31 0)
+			(effects
+				(font
+					(size 1.27 1.27)
+				)
+			)
+		)
+		(property "Footprint" "NetTie:NetTie-2_SMD_Pad0.5mm"
+			(at 45.72 69.85 0)
+			(effects
+				(font
+					(size 1.27 1.27)
+				)
+				(hide yes)
+			)
+		)
+		(property "Datasheet" "~"
+			(at 45.72 69.85 0)
+			(effects
+				(font
+					(size 1.27 1.27)
+				)
+				(hide yes)
+			)
+		)
+		(property "Description" "Net tie, 2 pins"
+			(at 45.72 69.85 0)
+			(effects
+				(font
+					(size 1.27 1.27)
+				)
+				(hide yes)
+			)
+		)
+		(pin "1"
+		)
+		(pin "2"
+		)
+		(instances
+			(project ""
+				(path "/ac1e7dc9-d098-4d7f-b836-51cfe621b1c8/f4117ea3-e4c6-4983-808a-c00237991f15"
+					(reference "NT1")
+					(unit 1)
+				)
